File: Kicad/Simply Split.kicad_pcb (KiCad board)
At the start: 2 copper layers, 284.7 x 99.7 mm, 74 parts, among them J1 Conn_01x02, SW1 SW_Push, SW11 SW_Push, SW13 SW_Push, SW15 SW_Push, SW17 SW_Push, SW19 SW_Push, SW21 SW_Push, SW23 SW_Push, SW25 SW_Push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

Commit message: Fixed repo as requested
Parts:
- removed the REF** at (203.5, 98.9)
Other:
- outline, holes or cut-outs redrawn
- board text removed: "${REFERENCE}"
Changed lines of the file:
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@@
 		)
 		(pad "1" thru_hole roundrect
-			(at 0 0 180)
-			(size 0.8 1.3)
-			(drill 0.5)
+			(at -0.1 0.2 180)
+			(size 1.2 1.4)
+			(drill 0.9)
 			(layers "*.Cu" "*.Mask")
 			(remove_unused_layers no)
@@
 		)
 		(pad "2" thru_hole oval
-			(at 1.25 0 180)
-			(size 0.8 1.3)
-			(drill 0.5)
+			(at 1.35 0.2 180)
+			(size 1.2 1.4)
+			(drill 0.9)
 			(layers "*.Cu" "*.Mask")
 			(remove_unused_layers no)
@@
 		(embedded_fonts no)
 	)
-	(footprint "PCM_marbastlib-choc:CHOCv1HOLE"
-		(layer "F.Cu")
-		(at 203.5 98.9)
-		(property "Reference" "REF**"
-			(at 0 -0.5 0)
-			(unlocked yes)
-			(layer "F.SilkS")
-			(effects
-				(font
-					(size 1 1)
-					(thickness 0.1)
-				)
-			)
-		)
-		(property "Value" "CHOCv1HOLE"
-			(at 0 1 0)
-			(unlocked yes)
-			(layer "F.Fab")
-			(hide yes)
-			(effects
-				(font
-					(size 1 1)
-					(thickness 0.15)
-				)
-			)
-		)
-		(property "Datasheet" ""
-			(at 0 0 0)
-			(unlocked yes)
-			(layer "F.Fab")
-			(hide yes)
-			(effects
-				(font
-					(size 1 1)
-					(thickness 0.15)
-				)
-			)
-		)
-		(property "Description" ""
-			(at 0 0 0)
-			(unlocked yes)
-			(layer "F.Fab")
-			(hide yes)
-			(effects
-				(font
-					(size 1 1)
-					(thickness 0.15)
-				)
-			)
-		)
-		(attr through_hole)
-		(fp_rect
-			(start -6.9 -6.9)
-			(end 6.9 6.9)
-			(stroke
-				(width 0.1)
-				(type solid)
-			)
-			(fill no)
-			(layer "Edge.Cuts")
-		)
-		(fp_text user "${REFERENCE}"
-			(at 0 2.5 0)
-			(unlocked yes)
-			(layer "F.Fab")
-			(effects
-				(font
-					(size 1 1)
-					(thickness 0.15)
-				)
-			)
-		)
-		(embedded_fonts no)
-	)
 	(footprint "kicad.mod:SW_PG1350_reversible"
 		(layer "F.Cu")
@@
 		)
 	)
+	(gr_line
+		(start 284.5 109.3)
+		(end 284.5 55.400138)
+		(stroke
+			(width 0.1)
+			(type solid)
+		)
+		(layer "Edge.Cuts")
+	)
 	(gr_arc
 		(start 26.1775 53.031049)
@@
 	(gr_arc
 		(start 262.196617 128.11475)
-		(mid 263.519829 128.49364)
+		(mid 263.51983 128.493642)
 		(end 264.44196 129.515463)
 		(stroke
@@
 	(gr_arc
 		(start 287.298188 143.585733)
-		(mid 286.334549 143.392543)
+		(mid 286.334547 143.392546)
 		(end 285.519833 142.842848)
 		(stroke
@@
 		(layer "Edge.Cuts")
 	)
+	(gr_arc
+		(start 287 111.8)
+		(mid 285.232233 111.067767)
+		(end 284.5 109.3)
+		(stroke
+			(width 0.1)
+			(type default)
+		)
+		(layer "Edge.Cuts")
+	)
 	(gr_line
 		(start 250.303457 51.190762)
@@
 	)
 	(gr_arc
+		(start 282 52.900138)
+		(mid 283.767754 53.632373)
+		(end 284.5 55.400138)
+		(stroke
+			(width 0.1)
+			(type default)
+		)
+		(layer "Edge.Cuts")
+	)
+	(gr_arc
 		(start 144.5715 138.716983)
 		(mid 143.839267 140.48475)
@@
 	(gr_arc
 		(start 246.864473 46.27975)
-		(mid 248.326225 46.751628)
+		(mid 248.326248 46.751613)
 		(end 249.236164 47.989126)
 		(stroke
@@
 		(layer "Edge.Cuts")
 	)
+	(gr_arc
+		(start 308.394 111.8)
+		(mid 310.161767 112.532233)
+		(end 310.894 114.3)
+		(stroke
+			(width 0.1)
+			(type default)
+		)
+		(layer "Edge.Cuts")
+	)
 	(gr_line
 		(start 227.763287 47.989126)
@@
 	)
 	(gr_line
-		(start 310.894 55.400138)
+		(start 310.894 114.3)
 		(end 310.894 141.085733)
 		(stroke
@@
 	(gr_arc
 		(start 195 109.899767)
-		(mid 193.232234 109.167534)
+		(mid 193.232245 109.167532)
 		(end 192.5 107.399767)
 		(stroke
@@
 	(gr_arc
 		(start 252.675147 52.900138)
-		(mid 251.213395 52.42826)
+		(mid 251.213365 52.428282)
 		(end 250.303457 51.190762)
 		(stroke
@@
 	(gr_arc
 		(start 249.000351 128.11475)
-		(mid 247.232584 127.382517)
+		(mid 247.232633 127.382497)
 		(end 246.500351 125.61475)
 		(stroke
@@
 	(gr_arc
 		(start 227.763287 47.989126)
-		(mid 228.673223 46.751619)
+		(mid 228.673213 46.751596)
 		(end 230.134977 46.27975)
 		(stroke
@@
 		(layer "Edge.Cuts")
 	)
-	(gr_arc
-		(start 308.394 52.900138)
-		(mid 310.161767 53.632371)
-		(end 310.894 55.400138)
+	(gr_line
+		(start 308.394 111.8)
+		(end 287 111.8)
 		(stroke
 			(width 0.1)
-			(type default)
+			(type solid)
 		)
 		(layer "Edge.Cuts")
@@
 	(gr_arc
 		(start 273.959601 132.199839)
-		(mid 274.923243 132.393024)
+		(mid 274.923241 132.393027)
 		(end 275.737956 132.942724)
 		(stroke
@@
 	(gr_line
 		(start 252.675147 52.900138)
-		(end 308.394 52.900138)
+		(end 282 52.900138)
 		(stroke
 			(width 0.1)
@@
 	(gr_arc
 		(start 267.003851 132.199839)
-		(mid 265.945301 131.896707)
+		(mid 265.945279 131.89672)
 		(end 265.207576 131.079268)
 		(stroke
@@
 	(gr_arc
 		(start 244.000351 109.899767)
-		(mid 245.768144 110.631984)
+		(mid 245.768126 110.631987)
 		(end 246.500351 112.399767)
 		(stroke
@@
 	(gr_arc
 		(start 310.894 141.085733)
-		(mid 310.161767 142.8535)
+		(mid 310.161755 142.853479)
 		(end 308.394 143.585733)
 		(stroke
@@
 	(gr_arc
 		(start 226.696107 51.190423)
-		(mid 225.786169 52.427922)
+		(mid 225.786171 52.427929)
 		(end 224.324416 52.899799)
 		(stroke
@@
 	(gr_arc
 		(start 192.5 55.399799)
-		(mid 193.232233 53.632032)
+		(mid 193.232233 53.632033)
 		(end 195 52.899799)
 		(stroke
@@
 		(layer "Edge.Cuts")
 	)
-	(gr_text "${REFERENCE}"
-		(at 203.5 101.4 0)
-		(layer "F.Fab")
-		(effects
-			(font
-				(size 1 1)
-				(thickness 0.15)
-			)
-		)
-	)
 	(segment
